Commit message: bug fix

File: kinova_controller/gen3_robotiq_2f_85.urdf (robot description, URDF)
Before this commit: robot gen3_robotiq_2f_85, 11 links, 10 joints
Links:
- removed link base_link
- removed link bracelet_link
- removed link end_effector_link
- removed link forearm_link
- removed link half_arm_1_link
- removed link half_arm_2_link
- removed link robotiq_arg2f_base_link
- removed link shoulder_link
- removed link spherical_wrist_1_link
- removed link spherical_wrist_2_link
- removed link tool_frame
- added link Base_Link, mass 1.697; collision mesh filename=package://kortex_description/arms/gen3/6dof/meshes/base_lin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; visual mesh filename=package://kortex_description/arms/gen3/6dof/meshes/base_lin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
- added link Bicep_Link, mass 1.262; collision mesh filename=package://kortex_description/arms/gen3/6dof/meshes/bicep_li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; visual mesh filename=package://kortex_description/arms/gen3/6dof/meshes/bicep_li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
- added link Bracelet_Link, mass 0.5; collision mesh filename=package://kortex_description/arms/gen3/6dof/meshes/bracelet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; visual mesh filename=package://kortex_description/arms/gen3/6dof/meshes/bracelet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
- added link EndEffector_Link, mass 0; collision mesh filename=package://kortex_description/arms/gen3/6dof/meshes/EndEffec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; visual mesh filename=package://kortex_description/arms/gen3/6dof/meshes/EndEffec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
- added link ForeArm_Link, mass 0.93; collision mesh filename=package://kortex_description/arms/gen3/6dof/meshes/forearm_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; visual mesh filename=package://kortex_description/arms/gen3/6dof/meshes/forearm_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
- added link Shoulder_Link, mass 1.377; collision mesh filename=package://kortex_description/arms/gen3/6dof/meshes/shoulder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; visual mesh filename=package://kortex_description/arms/gen3/6dof/meshes/shoulder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
- added link SphericalWrist1_Link, mass 0.6781; collision mesh filename=package://kortex_description/arms/gen3/6dof/meshes/spherica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; visual mesh filename=package://kortex_description/arms/gen3/6dof/meshes/spherica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
- added link SphericalWrist2_Link, mass 0.678; collision mesh filename=package://kortex_description/arms/gen3/6dof/meshes/spherica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; visual mesh filename=package://kortex_description/arms/gen3/6dof/meshes/spherica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
Joints:
- removed joint end_effector
- removed joint gripper_base_joint
- removed joint joint_1
- removed joint joint_2
- removed joint joint_3
- removed joint joint_4
- removed joint joint_5
- removed joint joint_6
- removed joint joint_7
- removed joint tool_frame_joint
- added joint Actuator1: type continuous, parent Base_Link, child Shoulder_Link, origin xyz=0 0 0.15643 rpy=-3.1416 0.0 0.0, axis 0 0 1, limit effort=39 velocity=0.8727
- added joint Actuator2: type revolute, parent Shoulder_Link, child Bicep_Link, origin xyz=0 0.005375 -0.12838 rpy=1.5708 0.0 0.0, axis 0 0 1, limit lower=-2.41 upper=2.41 effort=39 velocity=0.8727
- added joint Actuator3: type revolute, parent Bicep_Link, child ForeArm_Link, origin xyz=0 -0.41 0 rpy=3.1416 0 0, axis 0 0 1, limit lower=-2.66 upper=2.66 effort=39 velocity=0.8727
- added joint Actuator4: type continuous, parent ForeArm_Link, child SphericalWrist1_Link, origin xyz=0 0.20843 -0.006375 rpy=1.5708 0.0 0.0, axis 0 0 1, limit effort=9 velocity=0.8727
- added joint Actuator5: type revolute, parent SphericalWrist1_Link, child SphericalWrist2_Link, origin xyz=0 -0.00017505 -0.10593 rpy=-1.5708 0.0 0.0, axis 0 0 1, limit lower=-2.23 upper=2.23 effort=9 velocity=0.8727
- added joint Actuator6: type continuous, parent SphericalWrist2_Link, child Bracelet_Link, origin xyz=0 0.10593 -0.00017505 rpy=1.5708 0.0 0.0, axis 0 0 1, limit effort=9 velocity=0.8727
- added joint EndEffector: type fixed, parent Bracelet_Link, child EndEffector_Link, origin xyz=0 0 -0.061525 rpy=3.1416 0 -3.1416, axis 0 0 0

Commit message: try potential urdf

File: kinova_controller/gen3_robotiq_2f_85.urdf (robot description, URDF)
Before this commit: robot GEN3-6DOF_VISION_URDF_ARM_V01, 8 links, 7 joints
Links:
- removed link Base_Link
- added link base_link, mass 1.697; collision mesh filename=package://kortex_description/arms/gen3/6dof/meshes/base_lin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; visual mesh filename=package://kortex_description/arms/gen3/6dof/meshes/base_lin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
- added link realsense_color_optical_frame
- added link realsense_link
Joints:
- added joint realsense_mount_joint: type fixed, parent EndEffector_Link, child realsense_link, origin xyz=0.01 0.0 0.052 rpy=-1.57079632679 -1.57079632679 0.0
- added joint realsense_optical_joint: type fixed, parent realsense_link, child realsense_color_optical_frame, origin xyz=0 0 0 rpy=-1.57079632679 0 -1.57079632679
- joint Actuator1: parent Base_Link -> base_link

Commit message: full cide

File: kinova_controller/gen3_robotiq_2f_85.urdf (robot description, URDF)
Before this commit: robot GEN3-6DOF_VISION_URDF_ARM_V01, 10 links, 9 joints
Links:
- removed link realsense_color_optical_frame
Joints:
- removed joint realsense_optical_joint
